File: PCB/macropad.kicad_pcb (KiCad board)
At the start: 2 copper layers, 99.1 x 41.9 mm, 26 parts, among them SW1 SW_Push, SW11 RotaryEncoder_Switch, SW2 SW_Push, SW3 SW_Push, SW4 SW_Push, SW5 SW_Push, SW6 SW_Push, SW7 SW_Push, SW8 SW_Push, U1 MOUDLE-SEEEDUINO-XIAO

Commit message: added 3d models to the kicad project
Parts:
- SW2, SW3, SW4, SW5, SW6, SW7, SW8: footprint Library:SW_Cherry_MX_1.00u_PCB_with-3d -> vl_macropad:SW_Cherry_MX_1.00u_PCB
