File: PCB/macropad.kicad_sch (KiCad schematic)
At the start: 26 parts, among them SW1 SW_Push, SW11 RotaryEncoder_Switch, SW2 SW_Push, SW3 SW_Push, SW4 SW_Push, SW5 SW_Push, SW6 SW_Push, SW7 SW_Push, SW8 SW_Push, U1 MOUDLE-SEEEDUINO-XIAO

Commit message: added 3d models to the kicad project
Parts:
- SW2, SW3, SW4, SW5, SW6, SW7, SW8: footprint Library:SW_Cherry_MX_1.00u_PCB_with-3d -> vl_macropad:SW_Cherry_MX_1.00u_PCB
Changed lines of the file:
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@@
 			)
 		)
-		(property "Footprint" "Library:SW_Cherry_MX_1.00u_PCB_with-3d"
+		(property "Footprint" "vl_macropad:SW_Cherry_MX_1.00u_PCB"
 			(at 34.29 118.11 0)
 			(hide yes)
@@
 			)
 		)
-		(property "Footprint" "Library:SW_Cherry_MX_1.00u_PCB_with-3d"
+		(property "Footprint" "vl_macropad:SW_Cherry_MX_1.00u_PCB"
 			(at 85.09 118.11 0)
 			(hide yes)
@@
 			)
 		)
-		(property "Footprint" "Library:SW_Cherry_MX_1.00u_PCB_with-3d"
+		(property "Footprint" "vl_macropad:SW_Cherry_MX_1.00u_PCB"
 			(at 110.49 118.11 0)
 			(hide yes)
@@
 			)
 		)
-		(property "Footprint" "Library:SW_Cherry_MX_1.00u_PCB_with-3d"
+		(property "Footprint" "vl_macropad:SW_Cherry_MX_1.00u_PCB"
 			(at 85.09 92.71 0)
 			(hide yes)
@@
 			)
 		)
-		(property "Footprint" "Library:SW_Cherry_MX_1.00u_PCB_with-3d"
+		(property "Footprint" "vl_macropad:SW_Cherry_MX_1.00u_PCB"
 			(at 110.49 92.71 0)
 			(hide yes)
@@
 			)
 		)
-		(property "Footprint" "Library:SW_Cherry_MX_1.00u_PCB_with-3d"
+		(property "Footprint" "vl_macropad:SW_Cherry_MX_1.00u_PCB"
 			(at 59.69 92.71 0)
 			(hide yes)
@@
 			)
 		)
-		(property "Footprint" "Library:SW_Cherry_MX_1.00u_PCB_with-3d"
+		(property "Footprint" "vl_macropad:SW_Cherry_MX_1.00u_PCB"
 			(at 59.69 118.11 0)
 			(hide yes)
